File: hardware/kicad_project/Placa mcu/atmega328p_sch.kicad_sch (KiCad schematic)
At the start: 9 parts, among them J1 AVR-ISP-6, SW1 SW_Push, U1 ATMEGA328P, Y1 16MHz

Commit message: Placa MCU REV0 e readme
Connections:
- net AREV renamed AREF
Changed lines of the file:
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@@
 		)
 	)
-	(label "AREV"
+	(label "AREF"
 		(at 203.2 72.39 0)
 		(effects
@@
 		)
 	)
-	(label "AREV"
+	(label "AREF"
 		(at 166.37 72.39 0)
 		(effects
