File: hardware/kicad_project/Placa mcu/Condicionamento_PH_sch.kicad_sch (KiCad schematic)
At the start: 9 parts, among them J1 AVR-ISP-6, SW1 SW_Push, U1 ATMEGA328P, Y1 16MHz

Commit message: Esquematico modular
Parts:
- removed C2, C3: 100nF, symbol edd-dev-lib:C_CER_100N_PTH
- removed C4, C5: 22pF, symbol edd-dev-lib:C_CER_22P_PTH
- removed J1: AVR-ISP-6, symbol Connector:AVR-ISP-6
- removed SW1: SW_Push, symbol Switch:SW_Push
- removed U1: ATMEGA328P, Package_DIP:DIP-28_W7.62mm_LongPads, symbol edd-dev-lib:MCU_ATMEGA328P_DIP28
- removed Y1: 16MHz, symbol edd-dev-lib:XTAL_16MHZ_PTH
- added D1: 2,4V, symbol Device:D_Zener
- added J1: Conn_01x02, symbol Connector_Generic:Conn_01x02
- added R11: 10K, symbol Device:R
- added RV1: 10K, symbol Device:R_Potentiometer_Trim
- added RV3: 100K, symbol Device:R_Potentiometer_Trim
- added U1: MCP6002-xMS, symbol Amplifier_Operational:MCP6002-xMS
Connections:
- net +5V: now also U1.8 (V+)
- net GND: now also D1.2 (A), R11.1, U1.4 (V-)
- new net: R11.2, RV3.2, RV3.3, U1.6 (-)
- new net: RV1.2, RV1.3, U1.3 (+)
- new net: D1.1 (K), RV1.1
- new net PH+: J1.1 (Pin_1), U1.5 (+)
- new net PH-: J1.2 (Pin_2), U1.1, U1.2 (-)
- new net PH_AD: RV3.1, U1.7
- no-connect marks 15 -> 0
Other:
- company: Edson Almeida -> BAREMETAL
- title: Microcontrolador  -> (none)
